File: BeeWeight_MKRWAN_V4/BeeWeight_MKRWAN_V4.sch (KiCad schematic (older format))
At the start: 31 parts, among them J10 694103107102, J2 691412120004B, J3 691412120004B, J4 691412120004B, J5 691412120004B, J7 Conn_01x14_Female, J8 Conn_01x14_Female, J9 694108301002, Q1 IRLML6244, U1 ADS1241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

Commit message: Lundi soir : en cours de pin mapping
Parts:
- removed J9: 694108301002, USMB_Syl_Mont:Jack_DC_2.1mm Wurth_694108301002, symbol BeeWeight_MKRWAN-rescue:694108301002-Jack_DC_2.1mm_Wurth_694108301002
- added J1: SSW-120-01-X-S, SAMTEC_SSW-120-01-X-S, symbol SSW-120-01-X-S:SSW-120-01-X-S
- added J6: SSW-120-01-X-S, SSW-120-01-X-S:SAMTEC_SSW-120-01-X-S, symbol SSW-120-01-X-S:SSW-120-01-X-S
- added U3: LDL1117S50R, SOT230P700X180-4N, symbol LDL1117S33R:LDL1117S33R
Connections:
- net labels added: IO42_ALERT, IO42_CMD_MOS, IO42_CS, IO42_MISO, IO42_MOSI, IO42_SCL, IO42_SCLK, IO42_SDA, IO42_SHT_RST, IO42_VBAT
- wire segments 138 -> 142
- no-connect marks 16 -> 15
Other:
- note added: "LDO 3.3V"
- note removed: "Battery level measurement"
- note removed: "Supprimé"
- moved on the sheet: C16, J10, J7, J8
